Commit message: feat: Add the RGBD camera to the xacro and gazebo files

File: catkin_ws/src/my_robot/urdf/my_robot.xacro (robot description, xacro)
@@ -62,4 +62,10 @@
     <dynamics damping="1.0" friction="1.0"/>
   </joint>
+  <!--Joint RGB-D camera-->
+  <joint name="camera_optical_joint" type="fixed">
+    <origin xyz="0 0 0" rpy="-1.5707 0 -1.5707"/>
+    <parent link="camera_link"/>
+    <child link="camera_link_optical"/>
+  </joint>
   <!--Chasis model-->
   <link name='chassis'>
@@ -262,3 +268,6 @@
     </visual>
   </link>
+  <!--RGB-D camera link -->
+  <link name="camera_link_optical">
+  </link>
 </robot>

Commit message: fix: Correct the parent link of the RGBD Camera in the urdf file

File: catkin_ws/src/my_robot/urdf/my_robot.xacro (robot description, xacro)
@@ -65,5 +65,5 @@
   <joint name="camera_optical_joint" type="fixed">
     <origin xyz="0 0 0" rpy="-1.5707 0 -1.5707"/>
-    <parent link="camera_link"/>
+    <parent link="camera"/>
     <child link="camera_link_optical"/>
   </joint>
